File: Stir Plate.sch (EAGLE design)
At the start: 18 parts, among them IC1 555NEN, Q1 TIP31

Commit message: Correct Pot footprint / library entry
TODO: Fix board
Parts:
- R3: device Stir Plate:TRIM_US-RJ9W -> Stir Plate:TRIM_US-
Changed lines of the file:
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@@
 <part name="R1" library="Stir Plate" deviceset="R-US_" device="0207/10" value="1KR"/>
 <part name="R2" library="Stir Plate" deviceset="R-US_" device="0207/10" value="1kR"/>
-<part name="R3" library="Stir Plate" deviceset="TRIM_US-" device="RJ9W" value="10kR"/>
 <part name="C1" library="Stir Plate" deviceset="C-US" device="025-030X050" value="0.0047uF"/>
 <part name="C2" library="Stir Plate" deviceset="C-US" device="025-030X050" value="10000pF"/>
@@
 <part name="FRAME1" library="Stir Plate" deviceset="FRAME_A_L" device=""/>
 <part name="U$1" library="Stir Plate" deviceset="DOCFIELD" device=""/>
+<part name="R3" library="Stir Plate" deviceset="TRIM_US-" device="" value="10kR"/>
 </parts>
 <sheets>
@@
 <instance part="R1" gate="G$1" x="81.28" y="132.08" rot="R90"/>
 <instance part="R2" gate="G$1" x="180.34" y="106.68"/>
-<instance part="R3" gate="G$1" x="81.28" y="106.68" smashed="yes" rot="R270">
-<attribute name="NAME" x="71.12" y="104.14" size="1.778" layer="95"/>
-<attribute name="VALUE" x="71.12" y="101.6" size="1.778" layer="96"/>
-</instance>
 <instance part="C1" gate="G$1" x="93.98" y="88.9"/>
 <instance part="C2" gate="G$1" x="124.46" y="88.9" smashed="yes">
@@
 <instance part="FRAME1" gate="G$1" x="0" y="0"/>
 <instance part="U$1" gate="G$1" x="172.72" y="0"/>
+<instance part="R3" gate="G$1" x="81.28" y="106.68" smashed="yes" rot="R270">
+<attribute name="NAME" x="71.12" y="104.14" size="1.778" layer="95"/>
+<attribute name="VALUE" x="71.12" y="101.6" size="1.778" layer="96"/>
+</instance>
 </instances>
 <busses>
@@
 <segment>
 <pinref part="D3" gate="G$1" pin="A"/>
-<pinref part="R3" gate="G$1" pin="E"/>
 <wire x1="93.98" y1="111.76" x2="93.98" y2="106.68" width="0.1524" layer="91"/>
 <wire x1="93.98" y1="106.68" x2="88.9" y2="106.68" width="0.1524" layer="91"/>
+<pinref part="R3" gate="G$1" pin="E"/>
 </segment>
 </net>
@@
 <segment>
 <pinref part="D2" gate="G$1" pin="C"/>
-<pinref part="R3" gate="G$1" pin="A"/>
 <wire x1="68.58" y1="111.76" x2="68.58" y2="106.68" width="0.1524" layer="91"/>
 <wire x1="68.58" y1="106.68" x2="73.66" y2="106.68" width="0.1524" layer="91"/>
+<pinref part="R3" gate="G$1" pin="A"/>
 </segment>
 </net>
@@
 <net name="N$10" class="0">
 <segment>
-<pinref part="R3" gate="G$1" pin="S"/>
 <wire x1="81.28" y1="101.6" x2="81.28" y2="96.52" width="0.1524" layer="91"/>
 <wire x1="81.28" y1="96.52" x2="93.98" y2="96.52" width="0.1524" layer="91"/>
@@
 <wire x1="93.98" y1="91.44" x2="93.98" y2="96.52" width="0.1524" layer="91"/>
 <junction x="93.98" y="96.52"/>
-</segment>
-</net>
+<pinref part="R3" gate="G$1" pin="S"/>
+</segment>
+</net>
